File: Payload_Altimeter/COMPONENT_SHEETS/BAROMETER_MS5607-02.kicad_sch (KiCad schematic)
At the start: 2 parts, among them U7 MS5607-02BA

Commit message: Fixed Capacitor
Parts:
- C12: footprint Capacitor_Tantalum_SMD:CP_EIA-3528-15_AVX-H_Pad1.50x2.35mm_HandSolder -> Capacitor_SMD:C_0201_0603Metric
Changed lines of the file:
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@@
       (effects (font (size 1.27 1.27)) (justify left))
     )
-    (property "Footprint" "Capacitor_Tantalum_SMD:CP_EIA-3528-15_AVX-H_Pad1.50x2.35mm_HandSolder" (id 2) (at 162.2552 96.52 0)
+    (property "Footprint" "Capacitor_SMD:C_0201_0603Metric" (id 2) (at 162.2552 96.52 0)
       (effects (font (size 1.27 1.27)) hide)
     )

Commit message: Finished Schematic?
Connections:
- net PS is gone; now on net GND: U7.2 (PS)
- net ~{CSB} is gone; now on net GND: U7.4 (CSB), U7.5 (CSB)
- net +3V3 renamed 3v3
- net SDI_SDA renamed MOSI
- net SDO renamed MISO
Changed lines of the file:
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@@
     (comment 3 "Schematic depicting logical connections between components")
+  )
+  (junction (at 137.16 104.14) (diameter 0) (color 0 0 0 0)
   )
   (junction (at 161.29 81.28) (diameter 0) (color 0 0 0 0)
@@
   (junction (at 149.86 104.14) (diameter 0) (color 0 0 0 0)
   )
+  (wire (pts (xy 139.7 87.63) (xy 129.54 87.63))
+    (stroke (width 0) (type default) (color 0 0 0 0))
+  )
   (wire (pts (xy 149.86 81.28) (xy 161.29 81.28))
+    (stroke (width 0) (type default) (color 0 0 0 0))
+  )
+  (wire (pts (xy 137.16 104.14) (xy 149.86 104.14))
     (stroke (width 0) (type default) (color 0 0 0 0))
   )
@@
     (stroke (width 0) (type default) (color 0 0 0 0))
   )
+  (wire (pts (xy 129.54 87.63) (xy 129.54 104.14))
+    (stroke (width 0) (type default) (color 0 0 0 0))
+  )
   (polyline (pts (xy 171.45 71.12) (xy 171.45 119.38))
+    (stroke (width 0) (type default) (color 0 0 0 0))
+  )
+  (wire (pts (xy 139.7 97.79) (xy 137.16 97.79))
     (stroke (width 0) (type default) (color 0 0 0 0))
   )
@@
   )
   (wire (pts (xy 149.86 102.87) (xy 149.86 104.14))
+    (stroke (width 0) (type default) (color 0 0 0 0))
+  )
+  (wire (pts (xy 129.54 104.14) (xy 137.16 104.14))
+    (stroke (width 0) (type default) (color 0 0 0 0))
+  )
+  (wire (pts (xy 137.16 97.79) (xy 137.16 104.14))
     (stroke (width 0) (type default) (color 0 0 0 0))
   )
@@
     (effects (font (size 1.27 1.27)) (justify right))
   )
-  (hierarchical_label "SDO" (shape input) (at 139.7 90.17 180)
+  (hierarchical_label "MISO" (shape input) (at 139.7 90.17 180)
     (effects (font (size 1.27 1.27)) (justify right))
   )
-  (hierarchical_label "SDI_SDA" (shape input) (at 139.7 92.71 180)
-    (effects (font (size 1.27 1.27)) (justify right))
+  (hierarchical_label "3v3" (shape input) (at 161.29 80.01 90)
+    (effects (font (size 1.27 1.27)) (justify left))
   )
-  (hierarchical_label "PS" (shape input) (at 139.7 87.63 180)
-    (effects (font (size 1.27 1.27)) (justify right))
-  )
-  (hierarchical_label "~{CSB}" (shape input) (at 139.7 97.79 180)
+  (hierarchical_label "MOSI" (shape input) (at 139.7 92.71 180)
     (effects (font (size 1.27 1.27)) (justify right))
   )
@@
     (pin "8")
   )
-  (symbol (lib_id "Data_Collection_KiCAD_Project-rescue:+3.3V-power-Data_Collection_KiCAD_Project-rescue") (at 161.29 80.01 0) (unit 1)
-    (in_bom yes) (on_board yes)
-    (property "Reference" "#PWR041" (id 0) (at 161.29 83.82 0)
-      (effects (font (size 1.27 1.27)) hide)
-    )
-    (property "Value" "+3.3V" (id 1) (at 161.671 75.6158 0))
-    (property "Footprint" "" (id 2) (at 161.29 80.01 0)
-      (effects (font (size 1.27 1.27)) hide)
-    )
-    (property "Datasheet" "" (id 3) (at 161.29 80.01 0)
-      (effects (font (size 1.27 1.27)) hide)
-    )
-    (pin "1")
-  )
   (symbol (lib_id "Data_Collection_KiCAD_Project-rescue:GND-power-Data_Collection_KiCAD_Project-rescue") (at 149.86 105.41 0) (unit 1)
