File: Payload_Altimeter/COMPONENT_SHEETS/DSUB.kicad_sch (KiCad schematic)
At the start: 2 parts, among them J1 L717SDC37P1ACH4F

Commit message: added sd card
sd card was added and traces were placed for other components
Parts:
- removed JP1: 5V Disconnect, Jumper:SolderJumper-2_P1.3mm_Bridged_Pad1.0x1.5mm, symbol Jumper:SolderJumper_2_Bridged
Connections:
- net Dsub_5v is gone; now on net +5V: J1.20, J1.37
Other:
- note removed: "I have disconnected the 5V DSUB from the Data Collection because I do not want a situation to arise where the small linear regulator is powering the other boards on the bus. 5V on this board is only for usb power."
Changed lines of the file:
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@@
     (date "2021-12-06")
-  )
-  (wire (pts (xy 73.66 81.28) (xy 78.74 81.28))
-    (stroke (width 0) (type default) (color 0 0 0 0))
   )
   (wire (pts (xy 173.99 93.98) (xy 170.18 93.98))
     (stroke (width 0) (type default) (color 0 0 0 0))
   )
-  (wire (pts (xy 66.04 81.28) (xy 54.61 81.28))
-    (stroke (width 0) (type default) (color 0 0 0 0))
-  )
-  (text "I have disconnected the 5V DSUB from the Data Collection \nbecause I do not want a situation to arise where the small linear \nregulator is powering the other boards on the bus. 5V on this\n board is only for usb power."
-    (at 40.64 69.85 0)
-    (effects (font (size 1.27 1.27)) (justify left bottom))
-  )
-  (label "Dsub_5v" (at 144.78 48.26 180)
-    (effects (font (size 1.27 1.27)) (justify right bottom))
-  )
-  (label "Dsub_5v" (at 144.78 91.44 180)
-    (effects (font (size 1.27 1.27)) (justify right bottom))
-  )
-  (label "Dsub_5v" (at 78.74 81.28 0)
-    (effects (font (size 1.27 1.27)) (justify left bottom))
-  )
   (hierarchical_label "Alert_sda" (shape input) (at 144.78 58.42 180)
     (effects (font (size 1.27 1.27)) (justify right))
@@
     )
     (property "Datasheet" "" (id 3) (at 170.18 91.44 0)
-      (effects (font (size 1.27 1.27)) hide)
-    )
-    (pin "1")
-  )
-  (symbol (lib_id "Jumper:SolderJumper_2_Bridged") (at 69.85 81.28 0) (unit 1)
-    (in_bom yes) (on_board yes)
-    (property "Reference" "JP1" (id 0) (at 69.85 76.073 0))
-    (property "Value" "5V Disconnect" (id 1) (at 69.85 78.3844 0))
-    (property "Footprint" "Jumper:SolderJumper-2_P1.3mm_Bridged_Pad1.0x1.5mm" (id 2) (at 69.85 81.28 0)
-      (effects (font (size 1.27 1.27)) hide)
-    )
-    (property "Datasheet" "~" (id 3) (at 69.85 81.28 0)
-      (effects (font (size 1.27 1.27)) hide)
-    )
-    (pin "1")
-    (pin "2")
-  )
-  (symbol (lib_id "power:+5V") (at 54.61 81.28 0) (unit 1)
-    (in_bom yes) (on_board yes)
-    (property "Reference" "#PWR05" (id 0) (at 54.61 85.09 0)
-      (effects (font (size 1.27 1.27)) hide)
-    )
-    (property "Value" "+5V" (id 1) (at 54.991 76.8858 0))
-    (property "Footprint" "" (id 2) (at 54.61 81.28 0)
-      (effects (font (size 1.27 1.27)) hide)
-    )
-    (property "Datasheet" "" (id 3) (at 54.61 81.28 0)
       (effects (font (size 1.27 1.27)) hide)
     )
@@
       (effects (font (size 1.27 1.27)) hide)
     )
+    (pin "1")
+  )
+  (symbol (lib_id "power:+5V") (at 144.78 91.44 90) (unit 1)
+    (in_bom yes) (on_board yes) (fields_autoplaced)
+    (property "Reference" "#PWR0105" (id 0) (at 148.59 91.44 0)
+      (effects (font (size 1.27 1.27)) hide)
+    )
+    (property "Value" "+5V" (id 1) (at 141.6051 91.919 90)
+      (effects (font (size 1.27 1.27)) (justify left))
+    )
+    (property "Footprint" "" (id 2) (at 144.78 91.44 0)
+      (effects (font (size 1.27 1.27)) hide)
+    )
+    (property "Datasheet" "" (id 3) (at 144.78 91.44 0)
+      (effects (font (size 1.27 1.27)) hide)
+    )
+    (pin "1")
+  )
+  (symbol (lib_id "power:+5V") (at 144.78 48.26 0) (unit 1)
+    (in_bom yes) (on_board yes) (fields_autoplaced)
+    (property "Reference" "#PWR0104" (id 0) (at 144.78 52.07 0)
+      (effects (font (size 1.27 1.27)) hide)
+    )
+    (property "Value" "+5V" (id 1) (at 144.78 44.6555 0))
+    (property "Footprint" "" (id 2) (at 144.78 48.26 0)
+      (effects (font (size 1.27 1.27)) hide)
+    )
+    (property "Datasheet" "" (id 3) (at 144.78 48.26 0)
+      (effects (font (size 1.27 1.27)) hide)
+    )
